Commit message: add 3 ir camera sensor
Former-commit-id: ed0f66abfbb0ef15c34047df06869a138b166ad1

File: robot/turtlebot_follower.xacro (robot description, xacro)
@@ -14,5 +14,5 @@
   <stack_hexagons                 parent="base_link"/>
   <sensor_asus_xtion_pro          parent="base_link"/>
-	<link name="ir_led_link">
+  <link name="ir_led_link">
     <collision>
       <origin xyz="0 0 0" rpy="0 0 0"/>
@@ -34,5 +34,5 @@
     </inertial>
   </link>
-	<joint name="ir_led_joint" type="fixed">
+  <joint name="ir_led_joint" type="fixed">
     <axis xyz="0 1 0" />
     <origin xyz="0 0 0.025" rpy="0 0 0"/>
@@ -40,28 +40,31 @@
     <child link="ir_led_link"/>
   </joint>
-	<gazebo reference="ir_led_link">
-		<material>Gazebo/Red</material>
-	</gazebo>
-	<gazebo reference="ir_led_link">
-		<sensor type="ray" name="ir_led">
-			<pose>0 0 0 0 0 0</pose>
-			<visualize>true</visualize>
-			<update_rate>30</update_rate>
-			<ray>
-				<scan>
-					<horizontal>
-						<samples>10</samples>
-						<resolution>1</resolution>
-						<min_angle>-0.2</min_angle>
-						<max_angle>0.2</max_angle>
-					</horizontal>
-				</scan>
-				<range>
-					<min>0.01</min>
-					<max>2.0</max>
-					<resolution>0.01</resolution>
-				</range>
-			</ray>
-		</sensor>
-	</gazebo>
+  <gazebo reference="ir_led_link">
+    <material>Gazebo/Red</material>
+  </gazebo>
+  <gazebo reference="ir_led_link">
+<!--    <sensor type="ray" name="ir_led">
+      <pose>0 0 0 0 0 0</pose>
+      <visualize>true</visualize>
+      <update_rate>30</update_rate>
+      <ray>
+        <scan>
+          <horizontal>
+            <samples>10</samples>
+            <resolution>1</resolution>
+            <min_angle>-0.2</min_angle>
+            <max_angle>0.2</max_angle>
+          </horizontal>
+        </scan>
+        <range>
+          <min>0.01</min>
+          <max>2.0</max>
+          <resolution>0.01</resolution>
+        </range>
+      </ray>
+    </sensor>-->
+    <plugin name="ir_emitter" filename="libgazebo_ros_ir_emitter.so">
+     <frameName>ir_led_link</frameName>
+    </plugin>
+  </gazebo>
 </robot>

File: robot/turtlebot_guidance.xacro (robot description, xacro)
@@ -6,5 +6,5 @@
 -->
 <robot name="turtlebot" xmlns:xacro="http://ros.org/wiki/xacro">
-  <xacro:property name="cameraSize" value="0.05" />
+  <xacro:property name="cameraSize" value="0.03" />
   <xacro:include filename="$(find turtlebot_description)/urdf/turtlebot_common_library.urdf.xacro" />
   <xacro:include filename="$(find kobuki_description)/urdf/kobuki.urdf.xacro" />
@@ -14,5 +14,5 @@
   <stack_hexagons                 parent="base_link"/>
   <sensor_asus_xtion_pro          parent="base_link"/>
-  <link name="ir_camera_link">
+  <link name="ir_camera_link_mid">
     <collision>
       <origin xyz="0 0 0" rpy="0 0 0"/>
@@ -34,18 +34,76 @@
     </inertial>
   </link>
-  <joint name="ir_camera_joint" type="fixed">
+  <joint name="ir_camera_mid_joint" type="fixed">
     <axis xyz="0 1 0" />
-    <origin xyz="0.1 0 0.025" rpy="0 0 0"/>
+    <origin xyz="0.1 0 0.015" rpy="0 0 0"/>
     <parent link="plate_top_link"/>
-    <child link="ir_camera_link"/>
+    <child link="ir_camera_link_mid"/>
   </joint>
-  <gazebo reference="ir_camera_link">
+  <link name="ir_camera_link_l">
+    <collision>
+      <origin xyz="0 0 0" rpy="0 0 0"/>
+      <geometry>
+        <box size="${cameraSize} ${cameraSize} ${cameraSize}"/>
+      </geometry>
+    </collision>
+    <visual>
+      <origin xyz="0 0 0" rpy="0 0 0"/>
+      <geometry>
+        <box size="${cameraSize} ${cameraSize} ${cameraSize}"/>
+      </geometry>
+    </visual>
+    <inertial>
+      <mass value="0.1" />
+      <origin xyz="0 0 0" rpy="0 0 0"/>
+      <box_inertia m="${cameraSize}" x="${cameraSize}" y="${cameraSize}" z="${cameraSize}" />
+      <inertia ixx="1e-6" ixy="0" ixz="0" iyy="1e-6" iyz="0" izz="1e-6" />
+    </inertial>
+  </link>
+  <joint name="ir_camera_joint_l" type="fixed">
+    <axis xyz="0 1 0" />
+    <origin xyz="0.09 0.07 0.015" rpy="0 0 0.55"/>
+    <parent link="plate_top_link"/>
+    <child link="ir_camera_link_l"/>
+  </joint>
+  <link name="ir_camera_link_3">
+    <collision>
+      <origin xyz="0 0 0" rpy="0 0 0"/>
+      <geometry>
+        <box size="${cameraSize} ${cameraSize} ${cameraSize}"/>
+      </geometry>
+    </collision>
+    <visual>
+      <origin xyz="0 0 0" rpy="0 0 0"/>
+      <geometry>
+        <box size="${cameraSize} ${cameraSize} ${cameraSize}"/>
+      </geometry>
+    </visual>
+    <inertial>
+      <mass value="0.1" />
+      <origin xyz="0 0 0" rpy="0 0 0"/>
+      <box_inertia m="${cameraSize}" x="${cameraSize}" y="${cameraSize}" z="${cameraSize}" />
+      <inertia ixx="1e-6" ixy="0" ixz="0" iyy="1e-6" iyz="0" izz="1e-6" />
+    </inertial>
+  </link>
+  <joint name="ir_camera_joint_3" type="fixed">
+    <axis xyz="0 1 0" />
+    <origin xyz="0.09 -0.07 0.015" rpy="0 0 -0.55"/>
+    <parent link="plate_top_link"/>
+    <child link="ir_camera_link_3"/>
+  </joint>
+  <gazebo reference="ir_camera_link_mid">
     <material>Gazebo/Green</material>
   </gazebo>
-  <gazebo reference="ir_camera_link">
-    <sensor type="logical_camera" name="ir_camera">
+  <gazebo reference="ir_camera_link_l">
+    <material>Gazebo/Green</material>
+  </gazebo>
+  <gazebo reference="ir_camera_link_3">
+    <material>Gazebo/Green</material>
+  </gazebo>
+  <gazebo reference="ir_camera_link_mid">
+    <sensor type="logical_camera" name="ir_camera_mid">
       <always_on>true</always_on>
-      <visualize>false</visualize>
-      <update_rate>5.0</update_rate>
+      <visualize>true</visualize>
+      <update_rate>10.0</update_rate>
       <logical_camera>
         <near>0.05</near>
@@ -54,8 +112,44 @@
         <aspect_ratio>1.33</aspect_ratio>
       </logical_camera>
-      <plugin name="gazebo_ir_camera_plugin" filename="libgazebo_ros_ir_camera.so">
+      <plugin name="gazebo_ir_camera_mid_plugin" filename="libgazebo_ros_ir_camera.so">
         <robotNamespace>guidance</robotNamespace>
-        <topicName>/guidance/ir_camera/scan</topicName>
-        <frameName>ir_camera_link</frameName>
+        <topicName>/guidance/ir_camera_mid/scan</topicName>
+        <frameName>ir_camera_link_mid</frameName>
+      </plugin>
+    </sensor>
+  </gazebo>
+  <gazebo reference="ir_camera_link_l">
+    <sensor type="logical_camera" name="ir_camera_l">
+      <always_on>true</always_on>
+      <visualize>true</visualize>
+      <update_rate>10.0</update_rate>
+      <logical_camera>
+        <near>0.05</near>
+        <far>2.0</far>
+        <horizontal_fov>0.576</horizontal_fov>
+        <aspect_ratio>1.33</aspect_ratio>
+      </logical_camera>
+      <plugin name="gazebo_ir_camera_l_plugin" filename="libgazebo_ros_ir_camera.so">
+        <robotNamespace>guidance</robotNamespace>
+        <topicName>/guidance/ir_camera_l/scan</topicName>
+        <frameName>ir_camera_link_l</frameName>
+      </plugin>
+    </sensor>
+  </gazebo>
+  <gazebo reference="ir_camera_link_3">
+    <sensor type="logical_camera" name="ir_camera_3">
+      <always_on>true</always_on>
+      <visualize>true</visualize>
+      <update_rate>10.0</update_rate>
+      <logical_camera>
+        <near>0.05</near>
+        <far>2.0</far>
+        <horizontal_fov>0.576</horizontal_fov>
+        <aspect_ratio>1.33</aspect_ratio>
+      </logical_camera>
+      <plugin name="gazebo_ir_camera_r_plugin" filename="libgazebo_ros_ir_camera.so">
+        <robotNamespace>guidance</robotNamespace>
+        <topicName>/guidance/ir_camera_3/scan</topicName>
+        <frameName>ir_camera_link_3</frameName>
       </plugin>
     </sensor>

Commit message: add unit testing with spawn robot using service
Former-commit-id: 53c428a98110a2aa9536b2399e3f0d81500b290b

File: robot/turtlebot_follower.xacro (robot description, xacro)
@@ -10,5 +10,5 @@
   <xacro:include filename="$(find kobuki_description)/urdf/kobuki.urdf.xacro" />
   <xacro:include filename="$(find turtlebot_description)/urdf/stacks/hexagons.urdf.xacro"/>
-  <xacro:include filename="$(find turtlebot_description)/urdf/sensors/asus_xtion_pro.urdf.xacro"/>
+<!--  <xacro:include filename="$(find turtlebot_description)/urdf/sensors/asus_xtion_pro.urdf.xacro"/>-->
   <kobuki/>
   <stack_hexagons                 parent="base_link"/>
@@ -34,15 +34,16 @@
     </inertial>
   </link>
-  <joint name="ir_led_joint" type="fixed">
+  <joint name="ir_led_joint" type="revolute">
     <axis xyz="0 1 0" />
     <origin xyz="0 0 0.025" rpy="0 0 0"/>
     <parent link="plate_top_link"/>
     <child link="ir_led_link"/>
+    <limit lower="-0.01" upper="0.01" effort="0" velocity="0" />
   </joint>
   <gazebo reference="ir_led_link">
     <material>Gazebo/Red</material>
   </gazebo>
-  <gazebo reference="ir_led_link">
-<!--    <sensor type="ray" name="ir_led">
+  <gazebo reference="plate_top_link">
+    <sensor type="ray" name="ir_led">
       <pose>0 0 0 0 0 0</pose>
       <visualize>true</visualize>
@@ -63,8 +64,8 @@
         </range>
       </ray>
-    </sensor>-->
-    <plugin name="ir_emitter" filename="libgazebo_ros_ir_emitter.so">
+    </sensor>
+<!--    <plugin name="ir_emitter" filename="libgazebo_ros_ir_emitter.so">
      <frameName>ir_led_link</frameName>
-    </plugin>
+    </plugin>-->
   </gazebo>
 </robot>

File: robot/turtlebot_guidance.xacro (robot description, xacro)
@@ -40,5 +40,5 @@
     <child link="ir_camera_link_mid"/>
   </joint>
-  <link name="ir_camera_link_l">
+  <link name="l_ir_camera_link">
     <collision>
       <origin xyz="0 0 0" rpy="0 0 0"/>
@@ -64,7 +64,7 @@
     <origin xyz="0.09 0.07 0.015" rpy="0 0 0.55"/>
     <parent link="plate_top_link"/>
-    <child link="ir_camera_link_l"/>
+    <child link="l_ir_camera_link"/>
   </joint>
-  <link name="ir_camera_link_3">
+  <link name="r_ir_camera_link">
     <collision>
       <origin xyz="0 0 0" rpy="0 0 0"/>
@@ -86,23 +86,24 @@
     </inertial>
   </link>
-  <joint name="ir_camera_joint_3" type="fixed">
+  <joint name="r_ir_camera_joint" type="fixed">
     <axis xyz="0 1 0" />
     <origin xyz="0.09 -0.07 0.015" rpy="0 0 -0.55"/>
     <parent link="plate_top_link"/>
-    <child link="ir_camera_link_3"/>
+    <child link="r_ir_camera_link"/>
   </joint>
   <gazebo reference="ir_camera_link_mid">
     <material>Gazebo/Green</material>
   </gazebo>
-  <gazebo reference="ir_camera_link_l">
+  <gazebo reference="l_ir_camera_link">
     <material>Gazebo/Green</material>
   </gazebo>
-  <gazebo reference="ir_camera_link_3">
+  <gazebo reference="r_ir_camera_link">
     <material>Gazebo/Green</material>
   </gazebo>
   <gazebo reference="ir_camera_link_mid">
-    <sensor type="logical_camera" name="ir_camera_mid">
+    <sensor type="logical_camera" name="ir_camera_1">
       <always_on>true</always_on>
-      <visualize>true</visualize>
+      <visualize>false</visualize>
+      <topic>logical_camera_1/image</topic>
       <update_rate>10.0</update_rate>
       <logical_camera>
@@ -112,15 +113,16 @@
         <aspect_ratio>1.33</aspect_ratio>
       </logical_camera>
-      <plugin name="gazebo_ir_camera_mid_plugin" filename="libgazebo_ros_ir_camera.so">
+      <plugin name="ir_camera_controller" filename="libgazebo_ros_ir_camera.so">
         <robotNamespace>guidance</robotNamespace>
-        <topicName>/guidance/ir_camera_mid/scan</topicName>
+        <topicName>/scan</topicName>
         <frameName>ir_camera_link_mid</frameName>
       </plugin>
     </sensor>
   </gazebo>
-  <gazebo reference="ir_camera_link_l">
-    <sensor type="logical_camera" name="ir_camera_l">
+  <gazebo reference="l_ir_camera_link">
+    <sensor type="logical_camera" name="ir_camera_2 ">
       <always_on>true</always_on>
-      <visualize>true</visualize>
+      <visualize>false</visualize>
+      <topic>logical_camera_2/image</topic>
       <update_rate>10.0</update_rate>
       <logical_camera>
@@ -130,15 +132,16 @@
         <aspect_ratio>1.33</aspect_ratio>
       </logical_camera>
-      <plugin name="gazebo_ir_camera_l_plugin" filename="libgazebo_ros_ir_camera.so">
+      <plugin name="left_ir_camera_controller" filename="libgazebo_ros_ir_camera.so">
         <robotNamespace>guidance</robotNamespace>
-        <topicName>/guidance/ir_camera_l/scan</topicName>
-        <frameName>ir_camera_link_l</frameName>
+        <topicName>/scan</topicName>
+        <frameName>l_ir_camera_link</frameName>
       </plugin>
     </sensor>
   </gazebo>
-  <gazebo reference="ir_camera_link_3">
+  <gazebo reference="r_ir_camera_link">
     <sensor type="logical_camera" name="ir_camera_3">
       <always_on>true</always_on>
-      <visualize>true</visualize>
+      <visualize>false</visualize>
+      <topic>logical_camera_3/image</topic>
       <update_rate>10.0</update_rate>
       <logical_camera>
@@ -150,6 +153,6 @@
       <plugin name="gazebo_ir_camera_r_plugin" filename="libgazebo_ros_ir_camera.so">
         <robotNamespace>guidance</robotNamespace>
-        <topicName>/guidance/ir_camera_3/scan</topicName>
-        <frameName>ir_camera_link_3</frameName>
+        <topicName>/scan</topicName>
+        <frameName>r_ir_camera_link</frameName>
       </plugin>
     </sensor>
