Commit message: v0.3
Former-commit-id: cb92bfb6c20b2326b3ca9f1e8aa0249d16ff2339
Former-commit-id: 1bdc931a0d0821d6af25781cf5ec80367f27383d

File: turtlebot_guide_integration/robot/turtlebot_follower.xacro (robot description, xacro)
@@ -14,5 +14,5 @@
   <stack_hexagons                 parent="base_link"/>
   <sensor_asus_xtion_pro          parent="base_link"/>
-  <link name="ir_led_link">
+  <!--<link name="ir_led_link">
     <collision>
       <origin xyz="0 0 0" rpy="0 0 0"/>
@@ -65,7 +65,7 @@
       </ray>
     </sensor>
-<!--    <plugin name="ir_emitter" filename="libgazebo_ros_ir_emitter.so">
+    <plugin name="ir_emitter" filename="libgazebo_ros_ir_emitter.so">
      <frameName>ir_led_link</frameName>
-    </plugin>-->
-  </gazebo>
+    </plugin>
+  </gazebo>-->
 </robot>
