Commit message: v0.5
Former-commit-id: 2ee8ff74702d1a5e0cc99c298afcb57803350a50
Former-commit-id: c048eaafcc308c41b44b27f777ca8530a9c358c3

File: turtlebot_guide_integration/robot/turtlebot_guidance.xacro (robot description, xacro)
@@ -14,4 +14,12 @@
   <stack_hexagons                 parent="base_link"/>
   <sensor_asus_xtion_pro          parent="base_link"/>
+  <link name="laser_link">
+  </link>
+  <joint name="laser_joint" type="fixed">
+    <axis xyz="0 1 0" />
+    <origin xyz="0 0 0.015" rpy="0 0 0"/>
+    <parent link="plate_middle_link"/>
+    <child link="laser_link"/>
+  </joint>
   <link name="ir_camera_link_mid">
     <collision>
