Commit message: update the following rules

File: turtlebot_guide_execution/robot/tb_guide.xacro (robot description, xacro)
@@ -19,5 +19,5 @@
     <axis xyz="0 1 0" />
     <origin xyz="0 0 0.015" rpy="0 0 0"/>
-    <parent link="plate_middle_link"/>
+    <parent link="plate_bottom_link"/> <!-- middle -->
     <child link="laser_link"/>
   </joint>

Commit message: Fix local costmap not showing error

File: turtlebot_guide_execution/robot/tb_guide.xacro (robot description, xacro)
@@ -22,147 +22,3 @@
     <child link="laser_link"/>
   </joint>
-  <link name="ir_camera_link_mid">
-    <collision>
-      <origin xyz="0 0 0" rpy="0 0 0"/>
-      <geometry>
-        <box size="${cameraSize} ${cameraSize} ${cameraSize}"/>
-      </geometry>
-    </collision>
-    <visual>
-      <origin xyz="0 0 0" rpy="0 0 0"/>
-      <geometry>
-        <box size="${cameraSize} ${cameraSize} ${cameraSize}"/>
-      </geometry>
-    </visual>
-    <inertial>
-      <mass value="0.1" />
-      <origin xyz="0 0 0" rpy="0 0 0"/>
-      <box_inertia m="${cameraSize}" x="${cameraSize}" y="${cameraSize}" z="${cameraSize}" />
-      <inertia ixx="1e-6" ixy="0" ixz="0" iyy="1e-6" iyz="0" izz="1e-6" />
-    </inertial>
-  </link>
-  <joint name="ir_camera_mid_joint" type="fixed">
-    <axis xyz="0 1 0" />
-    <origin xyz="0.1 0 0.015" rpy="0 0 0"/>
-    <parent link="plate_top_link"/>
-    <child link="ir_camera_link_mid"/>
-  </joint>
-  <link name="l_ir_camera_link">
-    <collision>
-      <origin xyz="0 0 0" rpy="0 0 0"/>
-      <geometry>
-        <box size="${cameraSize} ${cameraSize} ${cameraSize}"/>
-      </geometry>
-    </collision>
-    <visual>
-      <origin xyz="0 0 0" rpy="0 0 0"/>
-      <geometry>
-        <box size="${cameraSize} ${cameraSize} ${cameraSize}"/>
-      </geometry>
-    </visual>
-    <inertial>
-      <mass value="0.1" />
-      <origin xyz="0 0 0" rpy="0 0 0"/>
-      <box_inertia m="${cameraSize}" x="${cameraSize}" y="${cameraSize}" z="${cameraSize}" />
-      <inertia ixx="1e-6" ixy="0" ixz="0" iyy="1e-6" iyz="0" izz="1e-6" />
-    </inertial>
-  </link>
-  <joint name="ir_camera_joint_l" type="fixed">
-    <axis xyz="0 1 0" />
-    <origin xyz="0.09 0.07 0.015" rpy="0 0 0.55"/>
-    <parent link="plate_top_link"/>
-    <child link="l_ir_camera_link"/>
-  </joint>
-  <link name="r_ir_camera_link">
-    <collision>
-      <origin xyz="0 0 0" rpy="0 0 0"/>
-      <geometry>
-        <box size="${cameraSize} ${cameraSize} ${cameraSize}"/>
-      </geometry>
-    </collision>
-    <visual>
-      <origin xyz="0 0 0" rpy="0 0 0"/>
-      <geometry>
-        <box size="${cameraSize} ${cameraSize} ${cameraSize}"/>
-      </geometry>
-    </visual>
-    <inertial>
-      <mass value="0.1" />
-      <origin xyz="0 0 0" rpy="0 0 0"/>
-      <box_inertia m="${cameraSize}" x="${cameraSize}" y="${cameraSize}" z="${cameraSize}" />
-      <inertia ixx="1e-6" ixy="0" ixz="0" iyy="1e-6" iyz="0" izz="1e-6" />
-    </inertial>
-  </link>
-  <joint name="r_ir_camera_joint" type="fixed">
-    <axis xyz="0 1 0" />
-    <origin xyz="0.09 -0.07 0.015" rpy="0 0 -0.55"/>
-    <parent link="plate_top_link"/>
-    <child link="r_ir_camera_link"/>
-  </joint>
-  <gazebo reference="ir_camera_link_mid">
-    <material>Gazebo/Green</material>
-  </gazebo>
-  <gazebo reference="l_ir_camera_link">
-    <material>Gazebo/Green</material>
-  </gazebo>
-  <gazebo reference="r_ir_camera_link">
-    <material>Gazebo/Green</material>
-  </gazebo>
-<!--  <gazebo reference="ir_camera_link_mid">
-    <sensor type="logical_camera" name="ir_camera_1">
-      <always_on>true</always_on>
-      <visualize>false</visualize>
-      <topic>logical_camera_1/image</topic>
-      <update_rate>10.0</update_rate>
-      <logical_camera>
-        <near>0.05</near>
-        <far>2.0</far>
-        <horizontal_fov>0.576</horizontal_fov>
-        <aspect_ratio>1.33</aspect_ratio>
-      </logical_camera>
-      <plugin name="ir_camera_controller" filename="libgazebo_ros_ir_camera.so">
-        <robotNamespace>guidance</robotNamespace>
-        <topicName>/scan</topicName>
-        <frameName>ir_camera_link_mid</frameName>
-      </plugin>
-    </sensor>
-  </gazebo>
-  <gazebo reference="l_ir_camera_link">
-    <sensor type="logical_camera" name="ir_camera_2 ">
-      <always_on>true</always_on>
-      <visualize>false</visualize>
-      <topic>logical_camera_2/image</topic>
-      <update_rate>10.0</update_rate>
-      <logical_camera>
-        <near>0.05</near>
-        <far>2.0</far>
-        <horizontal_fov>0.576</horizontal_fov>
-        <aspect_ratio>1.33</aspect_ratio>
-      </logical_camera>
-      <plugin name="left_ir_camera_controller" filename="libgazebo_ros_ir_camera.so">
-        <robotNamespace>guidance</robotNamespace>
-        <topicName>/scan</topicName>
-        <frameName>l_ir_camera_link</frameName>
-      </plugin>
-    </sensor>
-  </gazebo>
-  <gazebo reference="r_ir_camera_link">
-    <sensor type="logical_camera" name="ir_camera_3">
-      <always_on>true</always_on>
-      <visualize>false</visualize>
-      <topic>logical_camera_3/image</topic>
-      <update_rate>10.0</update_rate>
-      <logical_camera>
-        <near>0.05</near>
-        <far>2.0</far>
-        <horizontal_fov>0.576</horizontal_fov>
-        <aspect_ratio>1.33</aspect_ratio>
-      </logical_camera>
-      <plugin name="gazebo_ir_camera_r_plugin" filename="libgazebo_ros_ir_camera.so">
-        <robotNamespace>guidance</robotNamespace>
-        <topicName>/scan</topicName>
-        <frameName>r_ir_camera_link</frameName>
-      </plugin>
-    </sensor>
-  </gazebo>-->
 </robot>
